File: ws1/pcb/ver0.1/_saved_tinybot.sch (KiCad schematic (older format))
At the start: 18 parts, among them IC1 ATTINY84-P, P1 PWR, P2 PIN Breakout, P3 ICSP, U1 LD1117S33TR, U2 L293D

Commit message: working on schematic
Parts:
- C1: renamed from C?; footprint (none) -> Capacitors_ThroughHole:C_Disc_D3_P2.5
- C2: renamed from C?; footprint (none) -> Capacitors_ThroughHole:C_Radial_D5_L11_P2.5
- D1, D2, D3: footprint (none) -> LEDs:LED-5MM
- IC1: footprint DIP14 -> Housings_DIP:DIP-14_W7.62mm
- JP1: footprint (none) -> Capacitors_SMD:C_0402
- JP2: renamed from JP?; footprint (none) -> Pin_Headers:Pin_Header_Straight_1x02
- P1: footprint (none) -> Pin_Headers:Pin_Header_Straight_1x02
- P2: footprint (none) -> Pin_Headers:Pin_Header_Straight_1x12
- P3: footprint (none) -> Pin_Headers:Pin_Header_Straight_2x03
- P4, P5: renamed from P?; footprint (none) -> Pin_Headers:Pin_Header_Straight_1x02
- R1, R2, R3: footprint (none) -> Resistors_ThroughHole:Resistor_Horizontal_RM10mm
- U1: footprint SOT-223 -> Power_Integrations:TO-220
- U2: footprint (none) -> Housings_DIP:DIP-16_W7.62mm
Changed lines of the file:
@@
 F 0 "IC1" H 4850 5350 50  0000 C CNN
 F 1 "ATTINY84-P" H 6400 3850 50  0000 C CNN
-F 2 "DIP14" H 5700 4400 50  0000 C CIN
+F 2 "Housings_DIP:DIP-14_W7.62mm" H 5700 4400 50  0000 C CIN
 F 3 "" H 5700 4600 50  0000 C CNN
 	1    5700 4600
@@
 F 0 "D3" H 8800 4100 50  0000 C CNN
 F 1 "LED" H 8800 3900 50  0000 C CNN
-F 2 "" H 8800 4000 50  0000 C CNN
+F 2 "LEDs:LED-5MM" H 8800 4000 50  0001 C CNN
 F 3 "" H 8800 4000 50  0000 C CNN
 	1    8800 4000
@@
 F 0 "D1" H 3600 4400 50  0000 C CNN
 F 1 "RED LED" H 3600 4200 50  0000 C CNN
-F 2 "" H 3600 4300 50  0000 C CNN
+F 2 "LEDs:LED-5MM" H 3600 4300 50  0001 C CNN
 F 3 "" H 3600 4300 50  0000 C CNN
 	1    3600 4300
@@
 F 0 "U2" H 5750 1850 60  0000 C CNN
 F 1 "L293D" H 5750 2850 60  0000 C CNN
-F 2 "" H 5850 2350 60  0000 C CNN
+F 2 "Housings_DIP:DIP-16_W7.62mm" H 5850 2350 60  0001 C CNN
 F 3 "" H 5850 2350 60  0000 C CNN
 	1    5750 2350
@@
 F 0 "P3" H 8750 2650 50  0000 C CNN
 F 1 "ICSP" H 8750 2250 50  0000 C CNN
-F 2 "" H 8750 1250 50  0000 C CNN
+F 2 "Pin_Headers:Pin_Header_Straight_2x03" H 8750 1250 50  0001 C CNN
 F 3 "" H 8750 1250 50  0000 C CNN
 	1    8750 2450
@@
 F 0 "R2" V 8280 3700 50  0000 C CNN
 F 1 "330" V 8200 3700 50  0000 C CNN
-F 2 "" V 8130 3700 50  0000 C CNN
+F 2 "Resistors_ThroughHole:Resistor_Horizontal_RM10mm" V 8130 3700 50  0001 C CNN
 F 3 "" H 8200 3700 50  0000 C CNN
 	1    8200 3700
@@
 F 0 "R3" V 8280 4000 50  0000 C CNN
 F 1 "330" V 8200 4000 50  0000 C CNN
-F 2 "" V 8130 4000 50  0000 C CNN
+F 2 "Resistors_ThroughHole:Resistor_Horizontal_RM10mm" V 8130 4000 50  0001 C CNN
 F 3 "" H 8200 4000 50  0000 C CNN
 	1    8200 4000
@@
 $EndComp
 $Comp
-L GND #PWR6
+L GND #PWR01
 U 1 1 56DBB7D0
 P 5700 6500
-F 0 "#PWR6" H 5700 6250 50  0001 C CNN
+F 0 "#PWR01" H 5700 6250 50  0001 C CNN
 F 1 "GND" H 5700 6350 50  0000 C CNN
 F 2 "" H 5700 6500 50  0000 C CNN
@@
 $EndComp
 $Comp
-L PWR_FLAG #FLG1
+L PWR_FLAG #FLG02
 U 1 1 56DBB7F9
 P 5700 6300
-F 0 "#FLG1" H 5700 6395 50  0001 C CNN
+F 0 "#FLG02" H 5700 6395 50  0001 C CNN
 F 1 "PWR_FLAG" H 5700 6480 50  0000 C CNN
 F 2 "" H 5700 6300 50  0000 C CNN
@@
 F 0 "U1" H 2700 4300 50  0000 C CNN
 F 1 "LD1117S33TR" H 2700 4250 50  0000 C CNN
-F 2 "SOT-223" H 2700 4150 50  0000 C CNN
+F 2 "Power_Integrations:TO-220" H 2700 4150 50  0000 C CNN
 F 3 "" H 2700 4050 50  0000 C CNN
 	1    2700 4050
@@
 F 0 "P1" H 1500 4200 50  0000 C CNN
 F 1 "PWR" V 1600 4050 50  0000 C CNN
-F 2 "" H 1500 4050 50  0000 C CNN
+F 2 "Pin_Headers:Pin_Header_Straight_1x02" H 1500 4050 50  0001 C CNN
 F 3 "" H 1500 4050 50  0000 C CNN
 	1    1500 4050
@@
 F 0 "R1" V 3680 4950 50  0000 C CNN
 F 1 "330" V 3600 4950 50  0000 C CNN
-F 2 "" V 3530 4950 50  0000 C CNN
+F 2 "Resistors_ThroughHole:Resistor_Horizontal_RM10mm" V 3530 4950 50  0001 C CNN
 F 3 "" H 3600 4950 50  0000 C CNN
 	1    3600 4950
@@
 F 0 "D2" H 8800 3800 50  0000 C CNN
 F 1 "LED" H 8800 3600 50  0000 C CNN
-F 2 "" H 8800 3700 50  0000 C CNN
+F 2 "LEDs:LED-5MM" H 8800 3700 50  0001 C CNN
 F 3 "" H 8800 3700 50  0000 C CNN
 	1    8800 3700
@@
 F 0 "JP1" H 3600 5750 50  0000 C CNN
 F 1 "JUMPER" H 3600 5520 50  0000 C CNN
-F 2 "" H 3600 5600 50  0000 C CNN
+F 2 "Capacitors_SMD:C_0402" H 3600 5600 50  0001 C CNN
 F 3 "" H 3600 5600 50  0000 C CNN
 	1    3600 5600
@@
 $EndComp
 $Comp
-L GND #PWR1
+L GND #PWR03
 U 1 1 56DBBFEE
 P 1800 4400
-F 0 "#PWR1" H 1800 4150 50  0001 C CNN
+F 0 "#PWR03" H 1800 4150 50  0001 C CNN
 F 1 "GND" H 1800 4250 50  0000 C CNN
 F 2 "" H 1800 4400 50  0000 C CNN
@@
 VIN
 $Comp
-L GND #PWR3
+L GND #PWR04
 U 1 1 56DBC175
 P 3600 6100
-F 0 "#PWR3" H 3600 5850 50  0001 C CNN
+F 0 "#PWR04" H 3600 5850 50  0001 C CNN
 F 1 "GND" H 3600 5950 50  0000 C CNN
 F 2 "" H 3600 6100 50  0000 C CNN
@@
 $EndComp
 $Comp
-L GND #PWR9
+L GND #PWR05
 U 1 1 56DBC8EE
 P 9300 4100
-F 0 "#PWR9" H 9300 3850 50  0001 C CNN
+F 0 "#PWR05" H 9300 3850 50  0001 C CNN
 F 1 "GND" H 9300 3950 50  0000 C CNN
 F 2 "" H 9300 4100 50  0000 C CNN
@@
 $EndComp
 $Comp
-L GND #PWR4
+L GND #PWR06
 U 1 1 56DBCAAD
 P 4400 5300
-F 0 "#PWR4" H 4400 5050 50  0001 C CNN
+F 0 "#PWR06" H 4400 5050 50  0001 C CNN
 F 1 "GND" H 4400 5150 50  0000 C CNN
 F 2 "" H 4400 5300 50  0000 C CNN
@@
 $EndComp
 $Comp
-L GND #PWR2
+L GND #PWR07
 U 1 1 56DBCBAE
 P 2700 4600
-F 0 "#PWR2" H 2700 4350 50  0001 C CNN
+F 0 "#PWR07" H 2700 4350 50  0001 C CNN
 F 1 "GND" H 2700 4450 50  0000 C CNN
 F 2 "" H 2700 4600 50  0000 C CNN
@@
 $EndComp
 $Comp
-L GND #PWR5
+L GND #PWR08
 U 1 1 56DBCE29
 P 4700 2800
-F 0 "#PWR5" H 4700 2550 50  0001 C CNN
+F 0 "#PWR08" H 4700 2550 50  0001 C CNN
 F 1 "GND" H 4700 2650 50  0000 C CNN
 F 2 "" H 4700 2800 50  0000 C CNN
@@
 $EndComp
 $Comp
-L GND #PWR7
+L GND #PWR09
 U 1 1 56DBCE58
 P 6800 2800
-F 0 "#PWR7" H 6800 2550 50  0001 C CNN
+F 0 "#PWR09" H 6800 2550 50  0001 C CNN
 F 1 "GND" H 6800 2650 50  0000 C CNN
 F 2 "" H 6800 2800 50  0000 C CNN
@@
 VCC
 $Comp
-L GND #PWR8
+L GND #PWR010
 U 1 1 56DBDDBC
 P 9200 2700
-F 0 "#PWR8" H 9200 2450 50  0001 C CNN
+F 0 "#PWR010" H 9200 2450 50  0001 C CNN
 F 1 "GND" H 9200 2550 50  0000 C CNN
 F 2 "" H 9200 2700 50  0000 C CNN
@@
 F 0 "P2" H 7350 4050 50  0000 C CNN
 F 1 "PIN Breakout" V 7450 3400 50  0000 C CNN
-F 2 "" H 7350 3400 50  0000 C CNN
+F 2 "Pin_Headers:Pin_Header_Straight_1x12" H 7350 3400 50  0001 C CNN
 F 3 "" H 7350 3400 50  0000 C CNN
 	1    7350 3400
@@
 $EndComp
 $Comp
-L CONN_01X02 P?
+L CONN_01X02 P4
 U 1 1 56DBF2EA
 P 3900 2250
-F 0 "P?" H 3900 2400 50  0000 C CNN
+F 0 "P4" H 3900 2400 50  0000 C CNN
 F 1 "M1" V 4000 2250 50  0000 C CNN
-F 2 "" H 3900 2250 50  0000 C CNN
+F 2 "Pin_Headers:Pin_Header_Straight_1x02" H 3900 2250 50  0001 C CNN
 F 3 "" H 3900 2250 50  0000 C CNN
 	1    3900 2250
@@
 $EndComp
 $Comp
-L CONN_01X02 P?
+L CONN_01X02 P5
 U 1 1 56DBF569
 P 7700 2250
-F 0 "P?" H 7700 2400 50  0000 C CNN
+F 0 "P5" H 7700 2400 50  0000 C CNN
 F 1 "M2" V 7800 2250 50  0000 C CNN
-F 2 "" H 7700 2250 50  0000 C CNN
+F 2 "Pin_Headers:Pin_Header_Straight_1x02" H 7700 2250 50  0001 C CNN
 F 3 "" H 7700 2250 50  0000 C CNN
 	1    7700 2250
@@
 $EndComp
 $Comp
-L JUMPER JP?
+L JUMPER JP2
 U 1 1 56DBF9E9
 P 4300 1700
-F 0 "JP?" H 4300 1850 50  0000 C CNN
+F 0 "JP2" H 4300 1850 50  0000 C CNN
 F 1 "JUMPER" H 4300 1620 50  0000 C CNN
-F 2 "" H 4300 1700 50  0000 C CNN
+F 2 "Pin_Headers:Pin_Header_Straight_1x02" H 4300 1700 50  0001 C CNN
 F 3 "" H 4300 1700 50  0000 C CNN
 	1    4300 1700
@@
 DIR2B
 $Comp
-L C C?
+L C C1
 U 1 1 56DC0BCC
 P 2200 4350
-F 0 "C?" H 2225 4450 50  0000 L CNN
+F 0 "C1" H 2225 4450 50  0000 L CNN
 F 1 "0.1uF" H 2225 4250 50  0000 L CNN
-F 2 "" H 2238 4200 50  0000 C CNN
+F 2 "Capacitors_ThroughHole:C_Disc_D3_P2.5" H 2238 4200 50  0001 C CNN
 F 3 "" H 2200 4350 50  0000 C CNN
 	1    2200 4350
@@
 $EndComp
 $Comp
-L CP C?
+L CP C2
 U 1 1 56DC0D30
 P 3200 4350
-F 0 "C?" H 3225 4450 50  0000 L CNN
+F 0 "C2" H 3225 4450 50  0000 L CNN
 F 1 "10uF" H 3225 4250 50  0000 L CNN
-F 2 "" H 3238 4200 50  0000 C CNN
+F 2 "Capacitors_ThroughHole:C_Radial_D5_L11_P2.5" H 3238 4200 50  0001 C CNN
 F 3 "" H 3200 4350 50  0000 C CNN
 	1    3200 4350
@@
 $EndComp
 $Comp
-L GND #PWR?
+L GND #PWR011
 U 1 1 56DC0DFE
 P 2200 4600
-F 0 "#PWR?" H 2200 4350 50  0001 C CNN
+F 0 "#PWR011" H 2200 4350 50  0001 C CNN
 F 1 "GND" H 2200 4450 50  0000 C CNN
 F 2 "" H 2200 4600 50  0000 C CNN
@@
 $EndComp
 $Comp
-L GND #PWR?
+L GND #PWR012
 U 1 1 56DC0E3F
 P 3200 4600
-F 0 "#PWR?" H 3200 4350 50  0001 C CNN
+F 0 "#PWR012" H 3200 4350 50  0001 C CNN
 F 1 "GND" H 3200 4450 50  0000 C CNN
 F 2 "" H 3200 4600 50  0000 C CNN
